Commit message: Add inertials and velocity limits to emma description
MuJoCo rejects massless moving bodies, and none of the upstream links
had inertials. Add estimated masses to the arm (summing to the ~0.85 kg
spec), the gripper, and the base (3.6 kg, on a fixed base_inertia link
since the myAGV submodule can't be edited). Inertia tensors are solid
boxes over each link's mesh bounding box.

Every arm and gripper joint had velocity="0", which ros2_control can
treat as a hard limit. Set the arm to 2.79 rad/s (160 deg/s spec) and
the gripper to a 0.05 m/s placeholder.

File: src/emma_description/urdf/emma.urdf.xacro (robot description, xacro)
@@ -18,4 +18,18 @@
   <xacro:if value="${model in ['base', 'both']}">
     <xacro:include filename="$(find myagv_description)/urdf/myAGV.urdf"/>
+    <!-- Upstream myAGV links have no inertial, and the submodule can't be edited, so
+         the mass rides on a fixed child link. 3.6 kg is an estimate; the tensor is a
+         solid box over the base mesh bounds. -->
+    <link name="base_inertia">
+      <inertial>
+        <origin xyz="0.007 -0.0042 0.0661" rpy="0 0 0"/>
+        <mass value="3.6"/>
+        <inertia ixx="0.02098" ixy="0" ixz="0" iyy="0.0347" iyz="0" izz="0.04518"/>
+      </inertial>
+    </link>
+    <joint name="base_footprint_to_base_inertia" type="fixed">
+      <parent link="base_footprint"/>
+      <child link="base_inertia"/>
+    </joint>
   </xacro:if>
   <xacro:if value="${model in ['arm', 'both']}">

File: src/emma_description/urdf/mycobot_280_m5.urdf.xacro (robot description, xacro)
@@ -3,7 +3,12 @@
   myCobot 280 M5 arm, copied from elephantrobotics/mycobot_ros2 (d42ff61):
   mycobot_description/urdf/mycobot_280_m5/mycobot_280_m5.urdf
-  Only change: the g_base link has no visual or collision. Upstream draws the
-  optional G-base mounting plate there, which this robot does not have; the arm
-  bolts straight onto the myAGV. Meshes still load from mycobot_description.
+  Changes from upstream:
+  - The g_base link has no visual or collision. Upstream draws the optional G-base
+    mounting plate there, which this robot does not have; the arm bolts straight
+    onto the myAGV. Meshes still load from mycobot_description.
+  - Inertials added (upstream has none; MuJoCo rejects massless moving bodies).
+    Masses are estimates summing to the ~0.85 kg spec; the inertia tensors are
+    solid boxes over each mesh's bounding box. Not measured.
+  - Revolute velocity limits set to 2.79 rad/s (160 deg/s spec) instead of 0.
   BSD 2-Clause License
   Copyright (c) 2020, Elephant Robotics
@@ -31,4 +36,9 @@
   <link name="g_base"/>
   <link name="joint1">
+    <inertial>
+      <origin xyz="-0.0036 0 0.0365" rpy="0 0 0"/>
+      <mass value="0.25"/>
+      <inertia ixx="0.0002798" ixy="0" ixz="0" iyy="0.0003062" iyz="0" izz="0.000364"/>
+    </inertial>
     <visual>
       <geometry>
@@ -47,4 +57,9 @@
   </link>
   <link name="joint2">
+    <inertial>
+      <origin xyz="0 -0.0063 -0.0206" rpy="0 0 0"/>
+      <mass value="0.15"/>
+      <inertia ixx="0.0001407" ixy="0" ixz="0" iyy="0.0001236" iyz="0" izz="7.47e-05"/>
+    </inertial>
     <visual>
       <geometry>
@@ -61,4 +76,9 @@
   </link>
   <link name="joint3">
+    <inertial>
+      <origin xyz="-0.054 0 0.0576" rpy="0 0 0"/>
+      <mass value="0.1"/>
+      <inertia ixx="4.478e-05" ixy="0" ixz="0" iyy="0.0002284" iyz="0" izz="0.000222"/>
+    </inertial>
     <visual>
       <geometry>
@@ -75,4 +95,9 @@
   </link>
   <link name="joint4">
+    <inertial>
+      <origin xyz="-0.0468 0 0.0065" rpy="0 0 0"/>
+      <mass value="0.1"/>
+      <inertia ixx="4.339e-05" ixy="0" ixz="0" iyy="0.0001838" iyz="0" izz="0.0001715"/>
+    </inertial>
     <visual>
       <geometry>
@@ -91,4 +116,9 @@
   </link>
   <link name="joint5">
+    <inertial>
+      <origin xyz="0 -0.0084 -0.0073" rpy="0 0 0"/>
+      <mass value="0.08"/>
+      <inertia ixx="3.965e-05" ixy="0" ixz="0" iyy="2.845e-05" iyz="0" izz="3.106e-05"/>
+    </inertial>
     <visual>
       <geometry>
@@ -107,4 +137,9 @@
   </link>
   <link name="joint6">
+    <inertial>
+      <origin xyz="0 0.0067 -0.0094" rpy="0 0 0"/>
+      <mass value="0.07"/>
+      <inertia ixx="3.777e-05" ixy="0" ixz="0" iyy="2.762e-05" iyz="0" izz="2.736e-05"/>
+    </inertial>
     <visual>
       <geometry>
@@ -123,4 +158,9 @@
   </link>
   <link name="joint6_flange">
+    <inertial>
+      <origin xyz="0 0 -0.0052" rpy="0 0 0"/>
+      <mass value="0.02"/>
+      <inertia ixx="2.77e-06" ixy="0" ixz="0" iyy="2.77e-06" iyz="0" izz="4.915e-06"/>
+    </inertial>
     <visual>
       <geometry>
@@ -147,5 +187,5 @@
   <joint name="joint2_to_joint1" type="revolute">
     <axis xyz="0 0 1"/>
-    <limit effort = "1000.0" lower = "-2.9321" upper = "2.9321" velocity = "0"/>
+    <limit effort = "1000.0" lower = "-2.9321" upper = "2.9321" velocity = "2.79"/>
     <parent link="joint1"/>
     <child link="joint2"/>
@@ -154,5 +194,5 @@
   <joint name="joint3_to_joint2" type="revolute">
     <axis xyz="0 0 1"/>
-    <limit effort = "1000.0" lower = "-2.4434" upper = "2.4434" velocity = "0"/>
+    <limit effort = "1000.0" lower = "-2.4434" upper = "2.4434" velocity = "2.79"/>
     <parent link="joint2"/>
     <child link="joint3"/>
@@ -161,5 +201,5 @@
   <joint name="joint4_to_joint3" type="revolute">
     <axis xyz=" 0 0 1"/>
-    <limit effort = "1000.0" lower = "-2.6179" upper = "2.6179" velocity = "0"/>
+    <limit effort = "1000.0" lower = "-2.6179" upper = "2.6179" velocity = "2.79"/>
     <parent link="joint3"/>
     <child link="joint4"/>
@@ -168,5 +208,5 @@
   <joint name="joint5_to_joint4" type="revolute">
     <axis xyz=" 0 0 1"/>
-    <limit effort = "1000.0" lower = "-2.6179" upper = "2.6179" velocity = "0"/>
+    <limit effort = "1000.0" lower = "-2.6179" upper = "2.6179" velocity = "2.79"/>
     <parent link="joint4"/>
     <child link="joint5"/>
@@ -175,5 +215,5 @@
   <joint name="joint6_to_joint5" type="revolute">
     <axis xyz="0 0 1"/>
-    <limit effort = "1000.0" lower = "-2.7052" upper = "2.7925" velocity = "0"/>
+    <limit effort = "1000.0" lower = "-2.7052" upper = "2.7925" velocity = "2.79"/>
     <parent link="joint5"/>
     <child link="joint6"/>
@@ -182,5 +222,5 @@
   <joint name="joint6output_to_joint6" type="revolute">
     <axis xyz="0 0 1"/>
-    <limit effort = "1000.0" lower = "-3.14159" upper = "3.14159" velocity = "0"/>
+    <limit effort = "1000.0" lower = "-3.14159" upper = "3.14159" velocity = "2.79"/>
     <parent link="joint6"/>
     <child link="joint6_flange"/>

File: src/emma_description/urdf/parallel_gripper.urdf.xacro (robot description, xacro)
@@ -11,4 +11,6 @@
   - The mimic joint is named gripper_base_to_gripper_right; upstream called the
     right-finger joint gripper_base_to_gripper_left.
+  - Inertials added (estimated masses, bounding-box inertia) and the velocity limit
+    set to 0.05 m/s instead of 0. Neither is measured.
   gripper_controller is the left finger's travel in metres: 0 is open (15 mm between
   the fingertips), -0.007 is closed. The right finger mirrors it. The 7 mm travel is
@@ -16,6 +18,7 @@
 -->
 <robot xmlns:xacro="http://www.ros.org/wiki/xacro" name="parallel_gripper">
-  <xacro:macro name="gripper_link" params="name">
+  <xacro:macro name="gripper_link" params="name *inertial">
     <link name="${name}">
+      <xacro:insert_block name="inertial"/>
       <visual>
         <geometry>
@@ -30,7 +33,25 @@
     </link>
   </xacro:macro>
-  <xacro:gripper_link name="gripper_base"/>
-  <xacro:gripper_link name="gripper_left"/>
-  <xacro:gripper_link name="gripper_right"/>
+  <xacro:gripper_link name="gripper_base">
+    <inertial>
+      <origin xyz="0 -0.0095 -0.0035" rpy="0 0 0"/>
+      <mass value="0.05"/>
+      <inertia ixx="2.008e-05" ixy="0" ixz="0" iyy="2.942e-05" iyz="0" izz="2.697e-05"/>
+    </inertial>
+  </xacro:gripper_link>
+  <xacro:gripper_link name="gripper_left">
+    <inertial>
+      <origin xyz="0.016 0.003 0.0183" rpy="0 0 0"/>
+      <mass value="0.01"/>
+      <inertia ixx="3.418e-06" ixy="0" ixz="0" iyy="3.291e-06" iyz="0" izz="6.083e-07"/>
+    </inertial>
+  </xacro:gripper_link>
+  <xacro:gripper_link name="gripper_right">
+    <inertial>
+      <origin xyz="-0.016 0.003 0.0183" rpy="0 0 0"/>
+      <mass value="0.01"/>
+      <inertia ixx="3.418e-06" ixy="0" ixz="0" iyy="3.291e-06" iyz="0" izz="6.083e-07"/>
+    </inertial>
+  </xacro:gripper_link>
   <joint name="joint6_flange_to_gripper_base" type="fixed">
     <parent link="joint6_flange"/>
@@ -40,5 +61,5 @@
   <joint name="gripper_controller" type="prismatic">
     <axis xyz="1 0 0"/>
-    <limit effort="1000.0" lower="-0.007" upper="0.0" velocity="0"/>
+    <limit effort="1000.0" lower="-0.007" upper="0.0" velocity="0.05"/>
     <parent link="gripper_base"/>
     <child link="gripper_left"/>
@@ -46,5 +67,5 @@
   <joint name="gripper_base_to_gripper_right" type="prismatic">
     <axis xyz="1 0 0"/>
-    <limit effort="1000.0" lower="0.0" upper="0.007" velocity="0"/>
+    <limit effort="1000.0" lower="0.0" upper="0.007" velocity="0.05"/>
     <parent link="gripper_base"/>
     <child link="gripper_right"/>

Commit message: Add MuJoCo ros2_control block to emma description
A new ros2_control:=mujoco xacro argument adds a <ros2_control> block
using mujoco_ros2_control's MujocoSystemInterface, so the same URDF
serves both RViz and simulation. It exposes the six arm joints and the
gripper joint with position commands, and the mimic finger as state
only. The default (none) leaves the description unchanged.

File: src/emma_description/urdf/emma.urdf.xacro (robot description, xacro)
@@ -46,3 +46,41 @@
     </joint>
   </xacro:if>
+  <!-- ros2_control hardware: none (visualization only) or mujoco. The base is not
+       driven yet, so only the arm and gripper are exposed. -->
+  <xacro:arg name="ros2_control" default="none"/>
+  <!-- MJCF scene loaded by the MuJoCo hardware plugin. -->
+  <xacro:arg name="mujoco_model" default=""/>
+  <xacro:arg name="headless" default="false"/>
+  <xacro:macro name="position_joint" params="name">
+    <joint name="${name}">
+      <command_interface name="position"/>
+      <state_interface name="position">
+        <param name="initial_value">0.0</param>
+      </state_interface>
+      <state_interface name="velocity"/>
+    </joint>
+  </xacro:macro>
+  <xacro:if value="${'$(arg ros2_control)' == 'mujoco' and model == 'both'}">
+    <ros2_control name="MujocoSystem" type="system">
+      <hardware>
+        <plugin>mujoco_ros2_control/MujocoSystemInterface</plugin>
+        <param name="mujoco_model">$(arg mujoco_model)</param>
+        <param name="headless">$(arg headless)</param>
+      </hardware>
+      <xacro:position_joint name="joint2_to_joint1"/>
+      <xacro:position_joint name="joint3_to_joint2"/>
+      <xacro:position_joint name="joint4_to_joint3"/>
+      <xacro:position_joint name="joint5_to_joint4"/>
+      <xacro:position_joint name="joint6_to_joint5"/>
+      <xacro:position_joint name="joint6output_to_joint6"/>
+      <xacro:if value="${'$(arg gripper)' == 'parallel'}">
+        <xacro:position_joint name="gripper_controller"/>
+        <!-- Mimic finger: an MJCF equality constraint drives it, so it is state only. -->
+        <joint name="gripper_base_to_gripper_right">
+          <state_interface name="position"/>
+          <state_interface name="velocity"/>
+        </joint>
+      </xacro:if>
+    </ros2_control>
+  </xacro:if>
 </robot>

Commit message: Add mecanum wheel joints to emma description
The myAGV URDF has no wheels, and the submodule can't be edited, so
emma.urdf.xacro adds four wheel links with continuous joints about y.
Radius and centres are estimated from the myagv_base mesh, which sits
about 4 mm toward -y, hence the asymmetric y offsets. The links carry
inertia only: the base mesh already draws the wheels, and the MuJoCo
rollers are added during MJCF generation.

With ros2_control:=mujoco the wheels get a velocity command interface,
and a new pids_config_file argument passes the wheel velocity PID gains
to the MuJoCo hardware plugin.

File: src/emma_description/urdf/emma.urdf.xacro (robot description, xacro)
@@ -32,4 +32,28 @@
       <child link="base_inertia"/>
     </joint>
+    <!-- Mecanum wheels, added here because upstream has none. Geometry is estimated from the
+         myagv_base mesh, which also draws the wheels, so these links carry no visual. The
+         mesh sits about 4 mm toward -y, hence the asymmetric y. Mass is an estimate; the
+         tensor is a solid cylinder. MuJoCo's rollers come from postprocess_mjcf.py. -->
+    <xacro:property name="wheel_radius" value="0.04"/>
+    <xacro:macro name="mecanum_wheel" params="name x y">
+      <link name="${name}_wheel">
+        <inertial>
+          <mass value="0.1"/>
+          <inertia ixx="4.8e-5" ixy="0" ixz="0" iyy="8e-5" iyz="0" izz="4.8e-5"/>
+        </inertial>
+      </link>
+      <joint name="${name}_wheel_joint" type="continuous">
+        <parent link="base_footprint"/>
+        <child link="${name}_wheel"/>
+        <origin xyz="${x} ${y} ${wheel_radius}" rpy="0 0 0"/>
+        <axis xyz="0 1 0"/>
+        <limit effort="1000" velocity="30"/>
+      </joint>
+    </xacro:macro>
+    <xacro:mecanum_wheel name="front_left" x="0.1124" y="0.0945"/>
+    <xacro:mecanum_wheel name="front_right" x="0.1124" y="-0.1031"/>
+    <xacro:mecanum_wheel name="rear_left" x="-0.1014" y="0.0945"/>
+    <xacro:mecanum_wheel name="rear_right" x="-0.1014" y="-0.1031"/>
   </xacro:if>
   <xacro:if value="${model in ['arm', 'both']}">
@@ -46,9 +70,10 @@
     </joint>
   </xacro:if>
-  <!-- ros2_control hardware: none (visualization only) or mujoco. The base is not
-       driven yet, so only the arm and gripper are exposed. -->
+  <!-- ros2_control hardware: none (visualization only) or mujoco. -->
   <xacro:arg name="ros2_control" default="none"/>
   <!-- MJCF scene loaded by the MuJoCo hardware plugin. -->
   <xacro:arg name="mujoco_model" default=""/>
+  <!-- Velocity PID gains for the wheel motors, which MuJoCo drives by force. -->
+  <xacro:arg name="pids_config_file" default=""/>
   <xacro:arg name="headless" default="false"/>
   <xacro:macro name="position_joint" params="name">
@@ -61,4 +86,11 @@
     </joint>
   </xacro:macro>
+  <xacro:macro name="velocity_joint" params="name">
+    <joint name="${name}">
+      <command_interface name="velocity"/>
+      <state_interface name="position"/>
+      <state_interface name="velocity"/>
+    </joint>
+  </xacro:macro>
   <xacro:if value="${'$(arg ros2_control)' == 'mujoco' and model == 'both'}">
     <ros2_control name="MujocoSystem" type="system">
@@ -67,5 +99,10 @@
         <param name="mujoco_model">$(arg mujoco_model)</param>
         <param name="headless">$(arg headless)</param>
+        <param name="pids_config_file">$(arg pids_config_file)</param>
       </hardware>
+      <xacro:velocity_joint name="front_left_wheel_joint"/>
+      <xacro:velocity_joint name="front_right_wheel_joint"/>
+      <xacro:velocity_joint name="rear_left_wheel_joint"/>
+      <xacro:velocity_joint name="rear_right_wheel_joint"/>
       <xacro:position_joint name="joint2_to_joint1"/>
       <xacro:position_joint name="joint3_to_joint2"/>

Commit message: Start emma's arm folded back over the base in sim
Set initial_value on the arm joints. The gripper starts just inside its
open limit, since sitting exactly on it trips the joint limiter.

File: src/emma_description/urdf/emma.urdf.xacro (robot description, xacro)
@@ -77,9 +77,9 @@
   <xacro:arg name="pids_config_file" default=""/>
   <xacro:arg name="headless" default="false"/>
-  <xacro:macro name="position_joint" params="name">
+  <xacro:macro name="position_joint" params="name initial:=0.0">
     <joint name="${name}">
       <command_interface name="position"/>
       <state_interface name="position">
-        <param name="initial_value">0.0</param>
+        <param name="initial_value">${initial}</param>
       </state_interface>
       <state_interface name="velocity"/>
@@ -105,12 +105,14 @@
       <xacro:velocity_joint name="rear_left_wheel_joint"/>
       <xacro:velocity_joint name="rear_right_wheel_joint"/>
+      <!-- Starting pose: arm folded back over the base. -->
       <xacro:position_joint name="joint2_to_joint1"/>
-      <xacro:position_joint name="joint3_to_joint2"/>
-      <xacro:position_joint name="joint4_to_joint3"/>
-      <xacro:position_joint name="joint5_to_joint4"/>
+      <xacro:position_joint name="joint3_to_joint2" initial="2.259"/>
+      <xacro:position_joint name="joint4_to_joint3" initial="-2.505"/>
+      <xacro:position_joint name="joint5_to_joint4" initial="-0.495"/>
       <xacro:position_joint name="joint6_to_joint5"/>
       <xacro:position_joint name="joint6output_to_joint6"/>
       <xacro:if value="${'$(arg gripper)' == 'parallel'}">
-        <xacro:position_joint name="gripper_controller"/>
+        <!-- Just inside the open limit (0.0); exactly at it, drift trips the joint limiter. -->
+        <xacro:position_joint name="gripper_controller" initial="-0.0005"/>
         <!-- Mimic finger: an MJCF equality constraint drives it, so it is state only. -->
         <joint name="gripper_base_to_gripper_right">

Commit message: Add a wrist RGB-D camera to emma and a look pose for it
The gripper carries a box standing in for an Orbbec Gemini 305 on its +y side, looking along
the fingers and tilted 15 deg toward them, behind a camera:=gemini305 xacro argument (also on
display.launch.py). Its colour optical frame sits at the front face.

With the camera on, the folded start pose put it inside the upper arm, so joint 4 starts at
0.3 rad instead of -0.495 (HOME_Q and the ros2_control initial value). The planner ignores
camera-wrist pairs, and LOOK_Q points the camera at BLOCK_START from 0.2 m, 65 deg down;
test_look_pose re-solves it by IK and checks it sees the block and the place position.

File: src/emma_description/urdf/emma.urdf.xacro (robot description, xacro)
@@ -16,4 +16,6 @@
   <!-- End effector on the arm flange: parallel or none. Ignored without the arm. -->
   <xacro:arg name="gripper" default="parallel"/>
+  <!-- Wrist camera on the gripper: gemini305 or none. Ignored without the gripper. -->
+  <xacro:arg name="camera" default="gemini305"/>
   <xacro:if value="${model in ['base', 'both']}">
     <xacro:include filename="$(find myagv_description)/urdf/myAGV.urdf"/>
@@ -105,9 +107,10 @@
       <xacro:velocity_joint name="rear_left_wheel_joint"/>
       <xacro:velocity_joint name="rear_right_wheel_joint"/>
-      <!-- Starting pose: arm folded back over the base. -->
+      <!-- Starting pose: arm folded back over the base, wrist tipped up so the wrist camera
+           clears the upper arm. Keep in sync with HOME_Q in emma_manipulation. -->
       <xacro:position_joint name="joint2_to_joint1"/>
       <xacro:position_joint name="joint3_to_joint2" initial="2.259"/>
       <xacro:position_joint name="joint4_to_joint3" initial="-2.505"/>
-      <xacro:position_joint name="joint5_to_joint4" initial="-0.495"/>
+      <xacro:position_joint name="joint5_to_joint4" initial="0.3"/>
       <xacro:position_joint name="joint6_to_joint5"/>
       <xacro:position_joint name="joint6output_to_joint6"/>

File: src/emma_description/urdf/parallel_gripper.urdf.xacro (robot description, xacro)
@@ -80,3 +80,42 @@
     <origin xyz="0 0 0.045" rpy="0 0 0"/>
   </joint>
+  <!-- Wrist RGB-D camera, standing in for an Orbbec Gemini 305 (68 g, 23 x 42 x 42 mm). The mount
+       is a design choice, not a measured part: the body sits just past the +y edge of the
+       gripper_base mesh, looking along the fingers (gripper +z) and tilted 15 deg toward them so
+       the fingertips show at the bottom of the image, about 5 cm away (the minimum range is 4 cm).
+       wrist_camera_link follows REP 103 (x forward); its origin is the front face, where the
+       colour optical frame sits, so the sim camera does not render from inside the body. -->
+  <xacro:if value="${'$(arg camera)' == 'gemini305'}">
+    <link name="wrist_camera_link">
+      <inertial>
+        <origin xyz="-0.0115 0 0" rpy="0 0 0"/>
+        <mass value="0.068"/>
+        <inertia ixx="1.999e-05" ixy="0" ixz="0" iyy="1.299e-05" iyz="0" izz="1.299e-05"/>
+      </inertial>
+      <visual>
+        <origin xyz="-0.0115 0 0" rpy="0 0 0"/>
+        <geometry>
+          <box size="0.023 0.042 0.042"/>
+        </geometry>
+      </visual>
+      <collision>
+        <origin xyz="-0.0115 0 0" rpy="0 0 0"/>
+        <geometry>
+          <box size="0.023 0.042 0.042"/>
+        </geometry>
+      </collision>
+    </link>
+    <joint name="gripper_base_to_wrist_camera" type="fixed">
+      <parent link="gripper_base"/>
+      <child link="wrist_camera_link"/>
+      <origin xyz="0 0.037 0" rpy="0 -1.309 -1.5708"/>
+    </joint>
+    <!-- z forward, x right, y down in the image. -->
+    <link name="wrist_camera_color_optical_frame"/>
+    <joint name="wrist_camera_link_to_color_optical_frame" type="fixed">
+      <parent link="wrist_camera_link"/>
+      <child link="wrist_camera_color_optical_frame"/>
+      <origin xyz="0 0 0" rpy="-1.5708 0 -1.5708"/>
+    </joint>
+  </xacro:if>
 </robot>

Commit message: Add the base lidar's laser_frame to the URDF
Pose copied from upstream ydlidar_ros2_driver's static transform (8 cm up,
6.5 cm forward, facing -x). The regenerated MJCF gains a laser_frame site.

File: src/emma_description/urdf/emma.urdf.xacro (robot description, xacro)
@@ -58,4 +58,13 @@
     <xacro:mecanum_wheel name="rear_left" x="-0.1014" y="0.0945"/>
     <xacro:mecanum_wheel name="rear_right" x="-0.1014" y="-0.1031"/>
+    <!-- 2D lidar under the top plate. Frame name and pose are upstream's ydlidar_ros2_driver
+         launch (facing -x), not measured on this robot. MuJoCo's rangefinder fan is added by
+         postprocess_mjcf.py at this frame. -->
+    <link name="laser_frame"/>
+    <joint name="base_footprint_to_laser_frame" type="fixed">
+      <parent link="base_footprint"/>
+      <child link="laser_frame"/>
+      <origin xyz="0.065 0 0.08" rpy="0 0 ${pi}"/>
+    </joint>
   </xacro:if>
   <xacro:if value="${model in ['arm', 'both']}">
